Commit message: fix(piperx): extend zero-side IK limits and refine collision spheres
Allow J2 down to -3 degrees and J3 up to +3 degrees. Split eight conservative collision patches into 456 spheres while preserving surface coverage and collision-pair exclusions.

File: curobo/content/assets/robot/piper_x_description/urdf/piper_x_description.urdf (robot description, URDF)
Before this commit: robot piper_x, 7 links, 6 joints
Joints:
- joint joint2: limit lower=0 upper=3.1415926 effort=100 velocity=5 -> lower=-0.05235987755982989 upper=3.1415926 effort=100 velocity=5
- joint joint3: limit lower=-2.9670597 upper=0 effort=100 velocity=5 -> lower=-2.9670597 upper=0.05235987755982989 effort=100 velocity=5
